File: SWGenerator.kicad_sch (KiCad schematic)
At the start: 4 parts, among them J2 OLED, U2 CAT24C256, Y1 Si5351A-B-GT

Commit message: v0.2
Connections:
- net VCC: now also RP2040-zero1.3 (3v3), U2.8 (VCC), Y1.1 (VDD)
Changed lines of the file:
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@@
 	(wire
 		(pts
-			(xy 220.98 93.98) (xy 226.06 93.98)
-		)
-		(stroke
-			(width 0)
-			(type default)
-		)
-	)
-	(wire
-		(pts
-			(xy 161.29 80.01) (xy 167.64 80.01)
-		)
-		(stroke
-			(width 0)
-			(type default)
-		)
-	)
-	(wire
-		(pts
-			(xy 161.29 87.63) (xy 167.64 87.63)
+			(xy 220.98 93.98) (xy 224.79 93.98)
+		)
+		(stroke
+			(width 0)
+			(type default)
+		)
+	)
+	(wire
+		(pts
+			(xy 161.29 80.01) (xy 165.1 80.01)
+		)
+		(stroke
+			(width 0)
+			(type default)
+		)
+	)
+	(wire
+		(pts
+			(xy 161.29 87.63) (xy 165.1 87.63)
 		)
 		(stroke
@@
 	(wire
 		(pts
-			(xy 128.27 77.47) (xy 130.81 77.47)
+			(xy 123.19 77.47) (xy 130.81 77.47)
 		)
 		(stroke
@@
 	(wire
 		(pts
-			(xy 156.21 43.18) (xy 161.29 43.18)
+			(xy 156.21 43.18) (xy 160.02 43.18)
 		)
 		(stroke
@@
 	(wire
 		(pts
-			(xy 161.29 82.55) (xy 167.64 82.55)
-		)
-		(stroke
-			(width 0)
-			(type default)
-		)
-	)
-	(wire
-		(pts
-			(xy 161.29 77.47) (xy 167.64 77.47)
-		)
-		(stroke
-			(width 0)
-			(type default)
-		)
-	)
-	(wire
-		(pts
-			(xy 161.29 90.17) (xy 167.64 90.17)
-		)
-		(stroke
-			(width 0)
-			(type default)
-		)
-	)
-	(wire
-		(pts
-			(xy 220.98 83.82) (xy 226.06 83.82)
+			(xy 161.29 82.55) (xy 165.1 82.55)
+		)
+		(stroke
+			(width 0)
+			(type default)
+		)
+	)
+	(wire
+		(pts
+			(xy 161.29 77.47) (xy 165.1 77.47)
+		)
+		(stroke
+			(width 0)
+			(type default)
+		)
+	)
+	(wire
+		(pts
+			(xy 161.29 90.17) (xy 165.1 90.17)
+		)
+		(stroke
+			(width 0)
+			(type default)
+		)
+	)
+	(wire
+		(pts
+			(xy 220.98 83.82) (xy 224.79 83.82)
 		)
 		(stroke
@@
 	(wire
 		(pts
-			(xy 220.98 88.9) (xy 226.06 88.9)
+			(xy 220.98 88.9) (xy 224.79 88.9)
+		)
+		(stroke
+			(width 0)
+			(type default)
+		)
+	)
+	(wire
+		(pts
+			(xy 205.74 72.39) (xy 205.74 76.2)
 		)
 		(stroke
@@
 	(wire
 		(pts
-			(xy 156.21 45.72) (xy 161.29 45.72)
+			(xy 156.21 45.72) (xy 160.02 45.72)
 		)
 		(stroke
@@
 	(wire
 		(pts
-			(xy 161.29 74.93) (xy 167.64 74.93)
+			(xy 161.29 74.93) (xy 165.1 74.93)
 		)
 		(stroke
@@
 	(wire
 		(pts
-			(xy 161.29 85.09) (xy 167.64 85.09)
+			(xy 161.29 85.09) (xy 165.1 85.09)
 		)
 		(stroke
@@
 	)
 	(label "GP0"
-		(at 161.29 43.18 0)
+		(at 160.02 43.18 0)
 		(effects
 			(font
@@
 	)
 	(label "GP2"
-		(at 167.64 80.01 0)
+		(at 165.1 80.01 0)
 		(effects
 			(font
@@
 	)
 	(label "SCL"
-		(at 167.64 87.63 0)
+		(at 165.1 87.63 0)
 		(effects
 			(font
@@
 	)
 	(label "SDA"
-		(at 167.64 90.17 0)
+		(at 165.1 90.17 0)
+		(effects
+			(font
+				(size 1.27 1.27)
+			)
+			(justify left bottom)
+		)
+	)
+	(label "VCC"
+		(at 205.74 72.39 90)
 		(effects
 			(font
@@
 	)
 	(label "GP1"
-		(at 167.64 77.47 0)
+		(at 165.1 77.47 0)
 		(effects
 			(font
@@
 	)
 	(label "GP0"
-		(at 167.64 74.93 0)
-		(effects
-			(font
-				(size 1.27 1.27)
-			)
-			(justify left bottom)
+		(at 165.1 74.93 0)
+		(effects
+			(font
+				(size 1.27 1.27)
+			)
+			(justify left bottom)
+		)
+	)
+	(label "VCC"
+		(at 128.27 80.01 180)
+		(effects
+			(font
+				(size 1.27 1.27)
+			)
+			(justify right bottom)
 		)
 	)
 	(label "GP4"
-		(at 226.06 93.98 0)
+		(at 224.79 93.98 0)
 		(effects
 			(font
@@
 		)
 	)
+	(label "VCC"
+		(at 146.05 38.1 90)
+		(effects
+			(font
+				(size 1.27 1.27)
+			)
+			(justify left bottom)
+		)
+	)
 	(label "GP4"
-		(at 167.64 85.09 0)
+		(at 165.1 85.09 0)
 		(effects
 			(font
@@
 	)
 	(label "GP3"
-		(at 167.64 82.55 0)
+		(at 165.1 82.55 0)
 		(effects
 			(font
@@
 	)
 	(label "GP1"
-		(at 161.29 45.72 0)
+		(at 160.02 45.72 0)
 		(effects
 			(font
@@
 	)
 	(label "GP2"
-		(at 226.06 83.82 0)
+		(at 224.79 83.82 0)
 		(effects
 			(font
@@
 	)
 	(label "GP3"
-		(at 226.06 88.9 0)
+		(at 224.79 88.9 0)
 		(effects
 			(font
@@
 		(dnp no)
 		(property "Reference" "RP2040-zero1"
-			(at 146.05 72.136 0)
+			(at 146.304 71.882 0)
 			(effects
 				(font
@@
 		)
 		(property "Value" "~"
-			(at 146.05 72.39 0)
+			(at 146.05 73.152 0)
 			(effects
 				(font
@@
 	(symbol
 		(lib_id "power:GNDPWR")
-		(at 128.27 77.47 270)
+		(at 123.19 77.47 270)
 		(unit 1)
 		(exclude_from_sim no)
@@
 		(fields_autoplaced yes)
 		(property "Reference" "#PWR01"
+			(at 118.11 77.47 0)
+			(effects
+				(font
+					(size 1.27 1.27)
+				)
+				(hide yes)
+			)
+		)
+		(property "Value" "GNDPWR"
+			(at 119.38 77.3429 90)
+			(effects
+				(font
+					(size 1.27 1.27)
+				)
+				(justify right)
+			)
+		)
+		(property "Footprint" ""
+			(at 121.92 77.47 0)
+			(effects
+				(font
+					(size 1.27 1.27)
+				)
+				(hide yes)
+			)
+		)
+		(property "Datasheet" ""
+			(at 121.92 77.47 0)
+			(effects
+				(font
+					(size 1.27 1.27)
+				)
+				(hide yes)
+			)
+		)
+		(property "Description" "Power symbol creates a global label with name \"GNDPWR\" , global ground"
 			(at 123.19 77.47 0)
 			(effects
 				(font
-					(size 1.27 1.27)
-				)
-				(hide yes)
-			)
-		)
-		(property "Value" "GNDPWR"
-			(at 124.46 77.3429 90)
-			(effects
-				(font
-					(size 1.27 1.27)
-				)
-				(justify right)
-			)
-		)
-		(property "Footprint" ""
-			(at 127 77.47 0)
-			(effects
-				(font
-					(size 1.27 1.27)
-				)
-				(hide yes)
-			)
-		)
-		(property "Datasheet" ""
-			(at 127 77.47 0)
-			(effects
-				(font
-					(size 1.27 1.27)
-				)
-				(hide yes)
-			)
-		)
-		(property "Description" "Power symbol creates a global label with name \"GNDPWR\" , global ground"
-			(at 128.27 77.47 0)
-			(effects
-				(font
